File: bb60_v1/bb60_v1.kicad_sch (KiCad schematic)
At the start: 144 parts, among them J1 Conn_01x04, SW1 SW_Push, SW2 SW_Push, U1 STM32F072CBTx, U2 XC6206PxxxMR, U3 USBLC6-2SC6

Commit message: PCB Layout Rough Draft
Parts:
- removed D42, D63: 1N4148, Diode_THT:D_DO-35_SOD27_P7.62mm_Horizontal, symbol Diode:1N4148
- removed KC_BKSP1: MX_SW_solder, marbastlib-mx:SW_MX_1u, symbol marbastlib-mx:MX_SW_solder
- C1, C2, C3, C4, C5, C9: footprint (none) -> Capacitor_SMD:C_0201_0603Metric
- C6: footprint (none) -> Capacitor_SMD:C_0805_2012Metric
- C7, C8: value 10uF -> 1uF; footprint (none) -> Capacitor_SMD:C_0201_0603Metric
- D1, D10, D11, D12, D13, D14, D15, D16, D17, D18, D19, D2, D20, D21, D22, D23, D24, D25, D26, D27, D28, D29, D3, D30, D31, D32, D33, D34, D35, D36, D37, D38, D39, D4, D40, D41, D43, D44, D45, D46, D47, D48, D49, D5, D50, D51, D52, D53, D54, D55, D56, D57, D58, D59, D6, D60, D61, D62, D7, D8, D9: footprint Diode_THT:D_DO-35_SOD27_P7.62mm_Horizontal -> Diode_SMD:D_SOD-123
- KC_BKSP1: renamed from KC_BKSP; footprint marbastlib-mx:SW_MX_1u -> marbastlib-mx:STAB_MX_2u
- KC_BSLS1: renamed from KC_BSLS; footprint marbastlib-mx:SW_MX_1u -> marbastlib-mx:SW_MX_1.5u
- KC_CAPS1: renamed from KC_CAPS; footprint marbastlib-mx:SW_MX_1u -> marbastlib-mx:SW_MX_1.75u
- KC_ENT1: renamed from KC_ENT; footprint marbastlib-mx:SW_MX_1u -> Button_Switch_Keyboard:SW_Cherry_MX_2.25u_PCB
- KC_LALT1: renamed from KC_LALT; footprint marbastlib-mx:SW_MX_1u -> marbastlib-mx:SW_MX_1.5u
- KC_LCTL1: renamed from KC_LCTL; footprint marbastlib-mx:SW_MX_1u -> marbastlib-mx:SW_MX_1.5u
- KC_LSFT1: renamed from KC_LSFT; footprint marbastlib-mx:SW_MX_1u -> Button_Switch_Keyboard:SW_Cherry_MX_2.25u_PCB
- KC_RALT1: renamed from KC_RALT; footprint marbastlib-mx:SW_MX_1u -> marbastlib-mx:SW_MX_1.5u
- KC_RCTL1: renamed from KC_RCTL; footprint marbastlib-mx:SW_MX_1u -> marbastlib-mx:SW_MX_1.5u
- KC_SPC1: renamed from KC_SPC; footprint marbastlib-mx:SW_MX_1u -> marbastlib-mx:STAB_MX_7u
- KC_STEP1: renamed from KC_STEP; footprint marbastlib-mx:SW_MX_1u -> marbastlib-mx:SW_MX_1.75u_STP_1.25
- KC_TAB1: renamed from KC_TAB; footprint marbastlib-mx:SW_MX_1u -> marbastlib-mx:SW_MX_1.5u
- R1, R2, R3: footprint (none) -> Resistor_SMD:R_0201_0603Metric
- SW1, SW2: footprint (none) -> Button_Switch_SMD:SW_Push_1P1T_XKB_TS-1187A
- renumbered KC_A to KC_A1, KC_B to KC_B1, KC_C to KC_C1, KC_COMM to KC_COMM1, KC_D to KC_D1, KC_DOT to KC_DOT1, KC_E to KC_E1, KC_EQL to KC_EQL1, KC_ESC to KC_ESC1, KC_F to KC_F1, KC_G to KC_G1, KC_H to KC_H1, KC_I to KC_I1, KC_J to KC_J1, KC_K to KC_K1, KC_L to KC_L1, KC_LBRC to KC_LBRC1, KC_LGUI to KC_LGUI1, KC_M to KC_M1, KC_MINS to KC_MINS1, KC_N to KC_N1, KC_O to KC_O1, KC_P to KC_P1, KC_Q to KC_Q1, KC_QUOT to KC_QUOT1, KC_R to KC_R1, KC_RBRC to KC_RBRC1, KC_RGUI to KC_RGUI1, KC_RSFT to KC_RSFT1, KC_S to KC_S1, KC_SCLN to KC_SCLN1, KC_SLSH to KC_SLSH1, KC_T to KC_T1, KC_U to KC_U1, KC_V to KC_V1, KC_W to KC_W1, KC_X to KC_X1, KC_Y to KC_Y1, KC_Z to KC_Z1
Connections:
- net at D29.2 (A), KC_CAPS1.2: now also KC_STEP1.2

Commit message: Fixed stab keys on pcb
Parts:
- KC_BKSP1: footprint marbastlib-mx:STAB_MX_2u -> marbastlib-mx:SW_MX_1u
- KC_RSFT1: footprint marbastlib-mx:SW_MX_1u -> Button_Switch_Keyboard:SW_Cherry_MX_1.75u_PCB
- KC_SPC1: footprint marbastlib-mx:STAB_MX_7u -> marbastlib-mx:SW_MX_1u
Changed lines of the file:
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@@
 			)
 		)
-		(property "Footprint" "marbastlib-mx:STAB_MX_2u"
+		(property "Footprint" "marbastlib-mx:SW_MX_1u"
 			(at 246.38 36.83 0)
 			(hide yes)
@@
 			)
 		)
-		(property "Footprint" "marbastlib-mx:STAB_MX_7u"
+		(property "Footprint" "marbastlib-mx:SW_MX_1u"
 			(at 175.26 107.95 0)
 			(hide yes)
@@
 			)
 		)
-		(property "Footprint" "marbastlib-mx:SW_MX_1u"
+		(property "Footprint" "Button_Switch_Keyboard:SW_Cherry_MX_1.75u_PCB"
 			(at 236.22 90.17 0)
 			(hide yes)

Commit message: Added Ai03 Library, fixed stab positions
Parts:
- KC_ENT1, KC_LSFT1: footprint Button_Switch_Keyboard:SW_Cherry_MX_2.25u_PCB -> marbastlib-mx:SW_MX_1u
- KC_RSFT1: footprint Button_Switch_Keyboard:SW_Cherry_MX_1.75u_PCB -> marbastlib-mx:SW_MX_1u
Changed lines of the file:
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@@
 			)
 		)
-		(property "Footprint" "Button_Switch_Keyboard:SW_Cherry_MX_1.75u_PCB"
+		(property "Footprint" "marbastlib-mx:SW_MX_1u"
 			(at 236.22 90.17 0)
 			(hide yes)
@@
 			)
 		)
-		(property "Footprint" "Button_Switch_Keyboard:SW_Cherry_MX_2.25u_PCB"
+		(property "Footprint" "marbastlib-mx:SW_MX_1u"
 			(at 236.22 72.39 0)
 			(hide yes)
@@
 			)
 		)
-		(property "Footprint" "Button_Switch_Keyboard:SW_Cherry_MX_2.25u_PCB"
+		(property "Footprint" "marbastlib-mx:SW_MX_1u"
 			(at 114.3 90.17 0)
 			(hide yes)
