File: VP_Solder_KiCad/VP_Solder.kicad_pcb (KiCad board)
At the start: 2 copper layers, 281 x 94.4 mm, 168 parts, among them J1 Conn_01x04, SW1 SW_Push, SW2 SW_Push, U1 STM32F072CBTx, U2 XC6206PxxxMR, U3 USBLC6-2SC6

Commit message: added new footprints to custom library
Parts:
- removed G***: LOGO, LOGO
Other:
- board text removed: "Firmware:"

Commit message: updated schematic + pcb with new custom library symbols and footprints
Parts:
- removed REF**: STAB_MX_P_2u, marbastlib-mx:STAB_MX_P_2u
- removed REF** (x6): D_SOD-123, Diode_SMD:D_SOD-123
- removed REF** (x2): STAB_MX_P_2.25u, marbastlib-mx:STAB_MX_P_2.25u
- removed REF**: STAB_MX_P_7u, marbastlib-mx:STAB_MX_P_7u
- C1, C2, C3, C4, C5, C7, C8, C9: footprint Capacitor_SMD:C_0201_0603Metric -> shentobento:C_0201_0603Metric
- C6: footprint Capacitor_SMD:C_0805_2012Metric -> shentobento:C_0805_2012Metric
- COL0, COL1, COL10, COL11, COL12, COL13, COL2, COL3, COL4, COL5, COL6, COL7, COL8, COL9: footprint TestPoint:TestPoint_Pad_1.5x1.5mm -> shentobento:TestPoint_Pad_1.5x1.5mm
- D1, D10, D11, D12, D13, D14, D15, D16, D17, D18, D19, D2, D20, D21, D22, D23, D24, D25, D26, D27, D28, D29, D3, D30, D31, D32, D33, D34, D35, D36, D37, D38, D39, D4, D40, D41, D42, D43, D44, D45, D46, D47, D48, D49, D5, D50, D51, D52, D53, D54, D55, D56, D57, D58, D59, D6, D60, D61, D62, D7, D8, D9: footprint Diode_SMD:D_SOD-123 -> shentobento:D_SOD-123
- GND1: footprint TestPoint:TestPoint_Bridge_Pitch2.0mm_Drill0.7mm -> shentobento:TestPoint_Bridge_Pitch2.0mm_Drill0.7mm
- J1: footprint Connector_JST:JST_SH_SM04B-SRSS-TB_1x04-1MP_P1.00mm_Horizontal -> shentobento:JST_SH_1x04
- KC_0, KC_1, KC_2, KC_3, KC_4, KC_5, KC_6, KC_7, KC_8, KC_9, KC_A1, KC_B1, KC_BKSP1, KC_BKSP2, KC_BSLS2, KC_C1, KC_COMM1, KC_D1, KC_DOT1, KC_E1, KC_ENT1, KC_EQL1, KC_ESC1, KC_F1, KC_G1, KC_H1, KC_I1, KC_J1, KC_K1, KC_L1, KC_LBRC1, KC_LGUI1, KC_LSFT1, KC_M1, KC_MINS1, KC_MO1, KC_N1, KC_O1, KC_P1, KC_Q1, KC_QUOT1, KC_R1, KC_RBRC1, KC_RGUI1, KC_RSFT1, KC_S1, KC_SCLN1, KC_SLSH1, KC_SPC1, KC_T1, KC_U1, KC_V1, KC_W1, KC_X1, KC_Y1, KC_Z1: footprint marbastlib-mx:SW_MX_1u -> shentobento:SW_MX_1u
- KC_BSLS1, KC_LALT1, KC_LCTL1, KC_RALT1, KC_RCTL1, KC_TAB1: footprint marbastlib-mx:SW_MX_1.5u -> shentobento:SW_MX_1.5u
- KC_CAPS1: footprint marbastlib-mx:SW_MX_1.75u -> shentobento:SW_MX_1.75u
- KC_STEP1: footprint marbastlib-mx:SW_MX_1.75u_STP_1.25 -> shentobento:SW_MX_1.75u_STEPPED_1.25
- R1: footprint Resistor_SMD:R_0201_0603Metric -> shentobento:R_0201_0603Metric
- SW1, SW2: footprint Button_Switch_SMD:SW_Push_1P1T_XKB_TS-1187A -> shentobento:SW_Push_Reset_Bootloader
- U1: footprint Package_QFP:LQFP-48_7x7mm_P0.5mm -> shentobento:MCU_STM32F072CBTx
- U2: footprint Package_TO_SOT_SMD:SOT-23-3 -> shentobento:SOT-23-3
- U3: footprint Package_TO_SOT_SMD:SOT-23-6 -> shentobento:SOT-23-6
